File: t41_2_low_power_amplifier.kicad_pcb (KiCad board)
At the start: 2 copper layers, 70.1 x 66 mm, 57 parts, among them J1 5-1814832-1, J2 5-1814832-1, J3 B2B-XH-A_LF__SN_, J5 Screw_Terminal_01x02, Q1 Q_NPN_BCE, Q10 Q_NPN_BEC, Q4 Q_NPN_BCE, Q7 Q_NPN_BEC, Q8 Q_NPN_BEC, Q9 Q_NPN_BEC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

Commit message: Added Chernobyl device.
Parts:
- added R10: 56k, Resistor_SMD:R_1206_3216Metric, F.Cu at (152.9, 84.3)
- added R11: 2.2k, Resistor_SMD:R_1206_3216Metric, F.Cu at (153.0, 87.2)
- added U2: MCP9509HT-E/OT, footprints:SOT-23-5_MC_MCH, F.Cu at (152.9, 80.7)
- R14: value 47k -> 10k
- moved C11 11.3 mm to (112.6, 88.4), turned to 90 degrees
- moved R7 6.36 mm to (161.0, 81.7)
- moved FB1 6.36 mm to (157.3, 81.8)
- moved R14 2.75 mm to (112.6, 83.2)
Connections:
- C11 pad 2: /TXRX -> /SHDN_NOT
- R14 pad 2: GND -> /SHDN_NOT
- U1 pad 3: /TXRX -> /SHDN_NOT
- U3 pad 4: /TXRX -> /SHDN_NOT
Routing:
- net /SHDN_NOT: track 0.00 -> 59.1 mm, vias 0 -> 3
- net Net-(U1-VOUT): track 15.9 -> 23.0 mm
- net /10V_FINAL_REG: track 20.5 -> 16.8 mm
- net Net-(R10-Pad2): track 0.00 -> 2.93 mm
- net Net-(U2-SET): track 0.00 -> 2.67 mm
- net /TXRX: track 60.5 -> 62.1 mm, vias 2 -> 1
- net GND: vias 90 -> 93
Other:
- board text added: "T41-2 LOW POWER AMPLIFIER V1.6"
- board text removed: "T41-2 LOW POWER AMPLIFIER V1.5"
