File: t41_2_low_power_amplifier.kicad_pcb (KiCad board)
At the start: 2 copper layers, 70.1 x 66 mm, 60 parts, among them J1 5-1814832-1, J2 5-1814832-1, J3 B2B-XH-A_LF__SN_, J5 Screw_Terminal_01x02, Q1 Q_NPN_BCE, Q10 Q_NPN_BEC, Q4 Q_NPN_BCE, Q7 Q_NPN_BEC, Q8 Q_NPN_BEC, Q9 Q_NPN_BEC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

Commit message: Clean up for publish.
Parts:
- Q1, Q4: value Q_NPN_BCE -> Q_NPN_EBEC
- R11: value 2.2k -> 0
Routing:
- net /SHDN_NOT: vias 3 -> 2
