File: t41_2_low_power_amplifier.kicad_sch (KiCad schematic)
At the start: 56 parts, among them J1 5-1814832-1, J2 5-1814832-1, J3 B2B-XH-A_LF__SN_, J5 Screw_Terminal_01x02, Q1 Q_NPN_BCE, Q10 Q_NPN_BEC, Q4 Q_NPN_BCE, Q7 Q_NPN_BEC, Q8 Q_NPN_BEC, Q9 Q_NPN_BEC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

Commit message: Finishing up version 1.5.  Not ready for fab.
Parts:
- removed C9: 47uF, Capacitor_SMD:CP_Elec_6.3x5.7, symbol Device:C_Polarized_Small_US
- removed R27: 10, Resistor_SMD:R_1206_3216Metric, symbol Device:R_Small_US
- removed U2: MCP1804x-C002xOT, Package_TO_SOT_SMD:SOT-23-5, symbol Regulator_Linear:MCP1804x-C002xOT
- added C7, C8: 0.1uF, Capacitor_SMD:C_1206_3216Metric, symbol Device:C_Small
- added L1: ~, Binocular_Core:FT37-43, symbol InductorTapped:InductorTapped
- added U1: MCP1804T-A002I/MT, footprints:SOT-89_5MC_MCH, symbol MCP1804_SOT89:MCP1804T-A002I_MT
- C1: value 0.1uF -> 0.01uF
- C12, C20, C5: value 0.1uF -> 10uF
Connections:
- net 10V_FINAL_REG: now also L1.2; no longer T1.4 (SC)
- net 12V: now also FB2.1
- net GND: now also T1.4 (SC), U1.2 (GND)
- net TXRX: now also U1.3 (*SHDN)
- net at C6.1, FB1.1, R7.2: now also U1.1 (VOUT)
- net at C2.2, Q4.4 (C): now also C7.1, L1.1; no longer T1.3 (SA)
- net at C3.2, Q1.4 (C): now also C8.1, L1.3; no longer T1.5 (SB)
- net at C5.1, FB2.2: now also U1.5 (VIN)
- new net: C7.2, T1.3 (SA)
- new net: C8.2, T1.5 (SB)
Other:
- note added: "BN-43-302 4 TURNS BIFILAR #26 SECONDARY CENTER-TAPPED"
- note added: "BN-43-302 4 TURNS TRIFILAR #26"
- note added: "DNP = DO NOT PLACE"
- note added: "RF INPUT"
- note added: "RF OUTPUT"
- note removed: "BN-43-302 3 TURNS BIFILAR #26 SECONDARY CENTER-TAPPED"
- note removed: "BN-43-302 3 TURNS TRIFILAR #26"
- note removed: "INPUT"
- note removed: "OUTPUT"
- moved on the sheet: C12, C6, J1, T1

Commit message: Added Chernobyl device.
Parts:
- added R10: 56k, Resistor_SMD:R_1206_3216Metric, symbol Device:R_Small_US
- added R11: 2.2k, Resistor_SMD:R_1206_3216Metric, symbol Device:R_Small_US
- added U2: MCP9509HT-E/OT, footprints:SOT-23-5_MC_MCH, symbol MCP9509:MCP9509CT-E_OT
- R14: value 47k -> 10k
Connections:
- net GND: now also R11.2, U2.2 (GND), U2.4 (HYST); no longer R14.2
- net TXRX: now also U2.5 (VDD); no longer C11.2, U1.3 (*SHDN), U3.4 (~{SHDN})
- new net: R10.2, R11.1
- new net: R10.1, U2.1 (SET)
- new net SHDN_NOT: C11.2, R14.2, U1.3 (*SHDN), U2.3 (*OUT), U3.4 (~{SHDN})
Other:
- note added: "THERMOSTAT"
- moved on the sheet: J3, R14

Commit message: Clean up for publish.
Parts:
- Q1, Q4: value Q_NPN_BCE -> Q_NPN_EBEC
- Q10, Q7, Q8, Q9: symbol Device:Q_NPN_BEC -> Transistor_BJT:Q_NPN_BEC
- R11: value 2.2k -> 0
- U1: footprint footprints:SOT-89_5MC_MCH -> SOT-89_5MC_MCH
Other:
- note added: "10V REGULATOR SOT-23-5"
- note added: "10V REGULATOR SOT-89"
- note added: "FT37-43 8 TURNS BIFILAR #28"
- note added: "R11 CAN BE ADJUSTED TO SET THRESHOLD TEMPERATURE"
- note removed: "10V REGULATOR"
- moved on the sheet: C12, C7, C8, J1, L1, R10, R11, R14, T1
